File: sra_board_2022_kicad/sra_board_2022.kicad_sch (KiCad schematic)
At the start: 55 parts, among them J1 691131710004, J2 691131710004, SW1 DTS-6, SW2 DTS-6, SW3 DTS-6, SW4 DTS-6, U1 ESP32-DEVKITC-32D, X1 057-006-1

Commit message: Corrected Schematics for KiCad 6
Connections:
- net 0: now also JP4.3, POWER-JACK1.1
- net 12V_P: now also TB1.VM
- net 26: now also R5.2
- net AMS_IN: now also CIN1.2
- net OUT1A: now also TB1.A1
- net at L1.2, U$2.C: now also JP6.2
- no-connect marks 0 -> 4
Other:
- moved on the sheet: CIN2, CO2, D1, POWER-JACK1, R5, TB1, U$1
