File: sra_dev_board_2022/sra_dev_board_2022.kicad_pcb (KiCad board)
At the start: 2 copper layers, 81.2 x 91.5 mm, 110 parts, among them J1 Conn_01x19_Male, J11 Conn_01x05_Male, J12 Conn_01x05_Male, J13 Conn_01x05_Male, J2 Conn_01x03_Male, J3 Conn_01x03_Male, J4 Conn_01x03_Male, J5 Conn_01x19_Male, J6 DCJ200-10-A-XX-X_REVA, J7 Conn_01x06_Male, J8 Conn_01x06_Male, J9 Conn_01x04_Female, SW1 SW_Push_Dual, SW2 SW_Push_Dual, SW3 SW_Push_Dual, SW4 SW_Push_Dual, T1 Screw_Terminal_01x04, T2 Screw_Terminal_01x04, T3 Screw_Terminal_01x02, U1 ESP32-DEVKITC-32D, U2 AMS1117-3.3, U3 TB6612FNG, U4 TB6612FNG, U5 LM2576S-5

Commit message: Finalised SRA Dev Board 2022 Design, added gerbers, renders, assets
Parts:
- removed the kibuzzard-61F67ED2 at (79.8, 69.2)
- removed the kibuzzard-61F67ED2 at (89.5, 69.2)
- removed the kibuzzard-61F6808A at (72.6, 69.3)
- removed the kibuzzard-61F6808A at (82.4, 69.2)
- removed kibuzzard-61F68D30: G***, kibuzzard-61F68D30
- removed kibuzzard-61F6943B: G***, kibuzzard-61F6943B
- removed kibuzzard-61F6A95E: G***, kibuzzard-61F6A95E
- removed kibuzzard-61F6AA81: G***, kibuzzard-61F6AA81
- removed kibuzzard-61F6AC33: G***, kibuzzard-61F6AC33
- removed kibuzzard-61F6AC53: G***, kibuzzard-61F6AC53
- added G***: LOGO, logos:sra_logo_small_neg, F.Cu at (125.7, 75.6)
- added G***: LOGO, logos:sra_board_github_qr_code, F.Cu at (125.6, 99.9)
- added G***: LOGO, logos:sra_skull_small, F.Cu at (148.1, 71.9)
- added G***: LOGO, logos:sra_skull_big, B.Cu at (126.1, 62.3)
- added G***: LOGO, logos:pcb_power, B.Cu at (88.3, 49.5)
- added G***: LOGO, logos:sra_board_github_qr_code, B.Cu at (125.6, 99.9)
- added G***: LOGO, logos:sra_logo_small_neg, B.Cu at (125.7, 75.6)
- added REF**: Fiducial_0.75mm_Mask2.25mm, Fiducial:Fiducial_0.75mm_Mask2.25mm, F.Cu at (147.5, 115.3)
- added REF**: Fiducial_0.75mm_Mask2.25mm, Fiducial:Fiducial_0.75mm_Mask2.25mm, F.Cu at (78.0, 32.1)
- added REF**: KiCad-Logo2_5mm_SilkScreen, Symbol:KiCad-Logo2_5mm_SilkScreen, B.Cu at (88.2, 40.7)
- added REF**: OSHW-Logo2_9.8x8mm_SilkScreen, Symbol:OSHW-Logo2_9.8x8mm_SilkScreen, B.Cu at (95.3, 71.3)
- added kibuzzard-61F6A2E5: G***, kibuzzard-61F6A2E5, B.Cu at (141.2, 66.2)
- added kibuzzard-61F6A2FC: G***, kibuzzard-61F6A2FC, B.Cu at (143.9, 67.3)
- added kibuzzard-61F6A310: G***, kibuzzard-61F6A310, B.Cu at (146.4, 65.9)
- added kibuzzard-61F6A6E8: G***, kibuzzard-61F6A6E8, B.Cu at (149.7, 59.8)
- added kibuzzard-61F6A786: G***, kibuzzard-61F6A786, B.Cu at (149.9, 81.7)
- added kibuzzard-61F6ABAB: G***, kibuzzard-61F6ABAB, B.Cu at (149.6, 47.5)
- added kibuzzard-61F6AD1B: G***, kibuzzard-61F6AD1B, B.Cu at (125.3, 82.9)
- added kibuzzard-61F6AD42: G***, kibuzzard-61F6AD42, B.Cu at (125.2, 85.0)
- added kibuzzard-61F6B851: G***, kibuzzard-61F6B851, F.Cu at (72.6, 69.3)
- added kibuzzard-61F6B85D: G***, kibuzzard-61F6B85D, F.Cu at (79.8, 69.2)
- added kibuzzard-61F6B86D: G***, kibuzzard-61F6B86D, F.Cu at (82.4, 69.2)
- added kibuzzard-61F6B878: G***, kibuzzard-61F6B878, F.Cu at (89.5, 69.2)
- added kibuzzard-61F71050: G***, kibuzzard-61F71050, F.Cu at (75.8, 63.9)
- added kibuzzard-61F7105E: G***, kibuzzard-61F7105E, F.Cu at (86.0, 63.9)
- added kibuzzard-61F71139: G***, kibuzzard-61F71139, F.Cu at (126.0, 113.9)
- added kibuzzard-61F71139: G***, kibuzzard-61F71139, F.Cu at (125.9, 121.0)
- added kibuzzard-61F71200: G***, kibuzzard-61F71200, F.Cu at (70.8, 77.4)
- added kibuzzard-61F7127D: G***, kibuzzard-61F7127D, F.Cu at (70.8, 92.3)
- added kibuzzard-61F71294: G***, kibuzzard-61F71294, F.Cu at (70.8, 82.2)
- added kibuzzard-61F712A9: G***, kibuzzard-61F712A9, F.Cu at (70.8, 87.2)
- added kibuzzard-61F712DA: G***, kibuzzard-61F712DA, F.Cu at (70.8, 98.6)
- added kibuzzard-61F712EB: G***, kibuzzard-61F712EB, F.Cu at (70.8, 103.6)
- added kibuzzard-61F71302: G***, kibuzzard-61F71302, F.Cu at (70.8, 108.8)
- added kibuzzard-61F71318: G***, kibuzzard-61F71318, F.Cu at (70.8, 113.8)
- added kibuzzard-61F7147A: G***, kibuzzard-61F7147A, F.Cu at (70.9, 49.7)
- added kibuzzard-61F71491: G***, kibuzzard-61F71491, F.Cu at (70.9, 55.2)
- added kibuzzard-61F792D2: G***, kibuzzard-61F792D2, F.Cu at (146.4, 92.5)
- added kibuzzard-61F792D2: G***, kibuzzard-61F792D2, B.Cu at (146.8, 92.8)
- added kibuzzard-61F79319: G***, kibuzzard-61F79319, F.Cu at (147.7, 91.4)
- added kibuzzard-61F79319: G***, kibuzzard-61F79319, B.Cu at (147.9, 91.7)
- added kibuzzard-61F793BD: G***, kibuzzard-61F793BD, B.Cu at (148.1, 107.7)
- added kibuzzard-61F7B758: G***, kibuzzard-61F7B758, F.Cu at (116.4, 45.5)
- added kibuzzard-61F7BB7D: G***, kibuzzard-61F7BB7D, F.Cu at (110.5, 69.8)
- added kibuzzard-61F7C05B: G***, kibuzzard-61F7C05B, F.Cu at (136.4, 39.2)
- added kibuzzard-61F7C0C2: G***, kibuzzard-61F7C0C2, F.Cu at (105.6, 36.8)
- added kibuzzard-61F7C0CC: G***, kibuzzard-61F7C0CC, F.Cu at (147.3, 36.8)
- added kibuzzard-61F7C12E: G***, kibuzzard-61F7C12E, F.Cu at (116.5, 39.2)
- added kibuzzard-61F7C21A: G***, kibuzzard-61F7C21A, F.Cu at (132.2, 40.6)
- added kibuzzard-61F7C221: G***, kibuzzard-61F7C221, F.Cu at (129.4, 40.6)
- added kibuzzard-61F7C24F: G***, kibuzzard-61F7C24F, F.Cu at (137.5, 40.6)
- added kibuzzard-61F7C24F: G***, kibuzzard-61F7C24F, B.Cu at (137.5, 40.6)
- added kibuzzard-61F7CB17: G***, kibuzzard-61F7CB17, F.Cu at (126.3, 50.8)
- added kibuzzard-61F7D5C6: G***, kibuzzard-61F7D5C6, F.Cu at (126.5, 42.0)
- added kibuzzard-61F7D60F: G***, kibuzzard-61F7D60F, F.Cu at (138.1, 46.5)
- added kibuzzard-61F7D60F: G***, kibuzzard-61F7D60F, B.Cu at (138.1, 46.5)
- added kibuzzard-61F7D817: G***, kibuzzard-61F7D817, F.Cu at (97.2, 74.5)
- added kibuzzard-61F7D852: G***, kibuzzard-61F7D852, F.Cu at (102.1, 62.4)
- added kibuzzard-61F7E9C0: G***, kibuzzard-61F7E9C0, F.Cu at (90.6, 120.5)
- added kibuzzard-61F7EB28: G***, kibuzzard-61F7EB28, B.Cu at (126.2, 113.5)
- added kibuzzard-61F7EC33: G***, kibuzzard-61F7EC33, B.Cu at (140.9, 54.3)
- added kibuzzard-61F7EC75: G***, kibuzzard-61F7EC75, B.Cu at (143.8, 54.3)
- added kibuzzard-61F7EC8D: G***, kibuzzard-61F7EC8D, B.Cu at (147.1, 54.3)
- added kibuzzard-61F7ED72: G***, kibuzzard-61F7ED72, B.Cu at (105.6, 36.8)
- added kibuzzard-61F7ED8A: G***, kibuzzard-61F7ED8A, B.Cu at (147.3, 36.8)
- added kibuzzard-61F7EDAC: G***, kibuzzard-61F7EDAC, B.Cu at (129.4, 40.6)
- added kibuzzard-61F7EDC6: G***, kibuzzard-61F7EDC6, B.Cu at (132.2, 40.6)
- added kibuzzard-61F7EF48: G***, kibuzzard-61F7EF48, B.Cu at (136.3, 39.2)
- added kibuzzard-61F7EFEB: G***, kibuzzard-61F7EFEB, B.Cu at (116.3, 39.2)
- added kibuzzard-61F7F3F0: G***, kibuzzard-61F7F3F0, B.Cu at (126.5, 42.0)
- added kibuzzard-61F7F991: G***, kibuzzard-61F7F991, B.Cu at (126.3, 50.8)
- added kibuzzard-61F7FB1D: G***, kibuzzard-61F7FB1D, B.Cu at (111.2, 32.1)
- added kibuzzard-61F7FBA3: G***, kibuzzard-61F7FBA3, B.Cu at (73.4, 49.8)
- added kibuzzard-61F7FBC2: G***, kibuzzard-61F7FBC2, B.Cu at (73.4, 55.2)
- added kibuzzard-61F82282: G***, kibuzzard-61F82282, F.Cu at (148.7, 105.6)
- added kibuzzard-61F8332E: G***, kibuzzard-61F8332E, F.Cu at (76.2, 58.8)
- added kibuzzard-61F83333: G***, kibuzzard-61F83333, F.Cu at (86.0, 58.8)
- F1: footprint Diode_THT:D_DO-15_P5.08mm_Vertical_AnodeUp -> RUEF150_3,2A_trip:RUEF160
- F2: footprint Diode_THT:D_DO-15_P5.08mm_Vertical_AnodeUp -> RXEF050_1A_trip:RXEF050
- moved D10 47.0 mm to (97.0, 73.1), turned to 180 degrees
- moved R9 45.5 mm to (101.2, 73.1), turned to 0 degrees
- moved R10 41.0 mm to (98.5, 63.9), turned to 180 degrees
- moved D11 36.4 mm to (101.9, 63.9), turned to 0 degrees
- moved R15 3.02 mm to (95.0, 105.6)
- moved R16 2.98 mm to (98.0, 105.6)
- moved D8 2.34 mm to (135.2, 48.5)
- moved R8 2.34 mm to (135.2, 45.1)
- moved D7 1.93 mm to (132.7, 48.5)
- moved R7 1.93 mm to (132.7, 45.1)
- moved J7 1.75 mm to (122.9, 36.8)
- moved D6 1.53 mm to (130.2, 48.5)
- moved R6 1.53 mm to (130.2, 45.1)
- moved J8 1.29 mm to (129.9, 36.8)
- moved D5 1.15 mm to (127.7, 48.5)
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Connections:
- J8 pad 6: GND -> unconnected-(J8-Pad6)
- J9 pad 1: /3V3 -> GND
- J9 pad 2: GND -> /3V3
Routing:
- net /5V_P: track 168.9 -> 89.0 mm
- net /33: track 124.6 -> 89.1 mm
- net /32: track 92.0 -> 68.7 mm
- net /3V3: track 252.7 -> 239.7 mm, vias 3 -> 2
- net /14: track 123.1 -> 113.5 mm
- net /12: track 120.4 -> 111.5 mm
- net /21: track 64.8 -> 70.9 mm
- net Net-(R15-Pad2): track 4.87 -> 10.5 mm
- net /13: track 119.4 -> 114.4 mm
- net /22: track 52.1 -> 57.0 mm
- net /27: track 105.9 -> 110.4 mm
- net /16: track 58.0 -> 62.2 mm
- net /34: track 56.1 -> 59.6 mm
- net /4: track 65.0 -> 68.5 mm
- net GND: track 123.3 -> 119.9 mm
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Other:
- board size 81.2 x 91.5 mm -> 81.2 x 92.7 mm
- board text added: "0"
- board text added: "12"
- board text added: "13"
- board text added: "14"
- board text added: "15"
- board text added: "16"
- board text added: "17"
- board text added: "18"
- board text added: "19"
- board text added: "2"
- board text added: "21"
- board text added: "22"
- board text added: "23"
- board text added: "25"
- board text added: "26"
- board text added: "27"
- board text added: "3.3V"
- board text added: "32"
- board text added: "33"
- board text added: "34"
- board text added: "35"
- board text added: "36"
- board text added: "39"
- board text added: "4"
- board text added: "5"
- board text added: "5V"
- board text added: "CLK"
- board text added: "CMD"
- board text added: "Designed by"
- board text added: "EN"
- board text added: "GND"
- board text added: "IN1"
- board text added: "IN1=IN3=25, TP1 SHORT IN2=IN4=26, TP2 SHORT"
- board text added: "IN2"
- board text added: "IN3"
- board text added: "IN4"
- board text added: "IN5"
- board text added: "IN5=IN7=12, TP3 SHORT IN6=IN8=13, TP4 SHORT"
- board text added: "IN6"
- board text added: "IN7"
- board text added: "IN8"
- board text added: "M1A"
- board text added: "M1B"
- board text added: "M2A"
- board text added: "M2B"
- board text added: "M3A"
- board text added: "M3B"
- board text added: "M4A"
- board text added: "M4B"
- board text added: "PWM1"
- board text added: "PWM2"
- board text added: "PWM3"
- board text added: "PWM4"
- board text added: "Parallel Mode"
- board text added: "RX"
- board text added: "SD0"
- board text added: "SD1"
- board text added: "SD2"
- board text added: "SD3"
- board text added: "STBY"
- board text added: "TP1"
- board text added: "TP2"
- board text added: "TP3"
- board text added: "TP4"
- board text added: "TX"
- board text added: "VM"
