File: sra_dev_board_2022/sra_dev_board_2022.kicad_pcb (KiCad board)
At the start: 2 copper layers, 81.2 x 92.7 mm, 183 parts, among them J1 Conn_01x19_Male, J10 Conn_01x03_Male, J11 Conn_01x05_Male, J12 Conn_01x05_Male, J13 Conn_01x05_Male, J2 Conn_01x03_Male, J3 Conn_01x03_Male, J4 Conn_01x03_Male, J5 Conn_01x19_Male, J6 DCJ200-10-A-XX-X_REVA, J7 Conn_01x06_Male, J8 Conn_01x06_Male, J9 Conn_01x04_Female, SW1 SW_Push_Dual, SW2 SW_Push_Dual, SW3 SW_Push_Dual, SW4 SW_Push_Dual, T1 Screw_Terminal_01x04, T2 Screw_Terminal_01x04, T3 Screw_Terminal_01x02, U1 ESP32-DEVKITC-32D, U2 AMS1117-3.3, U3 TB6612FNG, U4 TB6612FNG, U5 LM2576S-5

Commit message: add DRV8825 Stepper Driver
Parts:
- removed R15, R16, R17, R18: 1k, Resistor_SMD:R_1206_3216Metric
- removed the REF** at (88.2, 40.7)
- removed the REF** at (95.3, 71.3)
- removed TB_A1, TB_B1: SW_Push_DPDT, dpdt_tht:dpdt_sw_2x03_tht
- removed TP1, TP2, TP3, TP4: TestPoint, testpoint_pad:pad_1,27-2,54_smd
- removed kibuzzard-61F67ED2 (x2): G***, kibuzzard-61F67ED2
- removed kibuzzard-61F6808A (x2): G***, kibuzzard-61F6808A
- removed kibuzzard-61F683BD (x4): G***, kibuzzard-61F683BD
- removed kibuzzard-61F6A036: G***, kibuzzard-61F6A036
- removed kibuzzard-61F6A04D: G***, kibuzzard-61F6A04D
- removed kibuzzard-61F6A06B: G***, kibuzzard-61F6A06B
- removed kibuzzard-61F6A088: G***, kibuzzard-61F6A088
- removed kibuzzard-61F6A2E5 (x2): G***, kibuzzard-61F6A2E5
- removed kibuzzard-61F6A6E8 (x2): G***, kibuzzard-61F6A6E8
- removed kibuzzard-61F6A786 (x2): G***, kibuzzard-61F6A786
- removed kibuzzard-61F6ABAB (x2): G***, kibuzzard-61F6ABAB
- removed kibuzzard-61F6AD1B (x2): G***, kibuzzard-61F6AD1B
- removed kibuzzard-61F6AD42 (x2): G***, kibuzzard-61F6AD42
- removed kibuzzard-61F6B851: G***, kibuzzard-61F6B851
- removed kibuzzard-61F6B85D: G***, kibuzzard-61F6B85D
- removed kibuzzard-61F6B86D: G***, kibuzzard-61F6B86D
- removed kibuzzard-61F6B878: G***, kibuzzard-61F6B878
- removed kibuzzard-61F71050: G***, kibuzzard-61F71050
- removed kibuzzard-61F7105E: G***, kibuzzard-61F7105E
- removed kibuzzard-61F71139 (x2): G***, kibuzzard-61F71139
- removed kibuzzard-61F71200: G***, kibuzzard-61F71200
- removed kibuzzard-61F7127D: G***, kibuzzard-61F7127D
- removed kibuzzard-61F71294: G***, kibuzzard-61F71294
- removed kibuzzard-61F712A9: G***, kibuzzard-61F712A9
- removed kibuzzard-61F712DA: G***, kibuzzard-61F712DA
- removed kibuzzard-61F712EB: G***, kibuzzard-61F712EB
- removed kibuzzard-61F71302: G***, kibuzzard-61F71302
- removed kibuzzard-61F71318: G***, kibuzzard-61F71318
- removed kibuzzard-61F7147A: G***, kibuzzard-61F7147A
- removed kibuzzard-61F71491: G***, kibuzzard-61F71491
- removed kibuzzard-61F792D2 (x2): G***, kibuzzard-61F792D2
- removed kibuzzard-61F79319 (x2): G***, kibuzzard-61F79319
- removed kibuzzard-61F793BD: G***, kibuzzard-61F793BD
- removed kibuzzard-61F7BB7D: G***, kibuzzard-61F7BB7D
- removed kibuzzard-61F7C05B: G***, kibuzzard-61F7C05B
- removed kibuzzard-61F7C0C2: G***, kibuzzard-61F7C0C2
- removed kibuzzard-61F7C0CC: G***, kibuzzard-61F7C0CC
- removed kibuzzard-61F7C12E: G***, kibuzzard-61F7C12E
- removed kibuzzard-61F7C21A: G***, kibuzzard-61F7C21A
- removed kibuzzard-61F7C221: G***, kibuzzard-61F7C221
- removed kibuzzard-61F7C24F (x2): G***, kibuzzard-61F7C24F
- removed kibuzzard-61F7CB17: G***, kibuzzard-61F7CB17
- removed kibuzzard-61F7D5C6: G***, kibuzzard-61F7D5C6
- removed kibuzzard-61F7D60F: G***, kibuzzard-61F7D60F
- removed kibuzzard-61F7D817: G***, kibuzzard-61F7D817
- removed kibuzzard-61F7D852: G***, kibuzzard-61F7D852
- removed kibuzzard-61F7EB28: G***, kibuzzard-61F7EB28
- removed kibuzzard-61F7EC33: G***, kibuzzard-61F7EC33
- removed kibuzzard-61F7EC75: G***, kibuzzard-61F7EC75
- removed kibuzzard-61F7EC8D: G***, kibuzzard-61F7EC8D
- removed kibuzzard-61F7ED72: G***, kibuzzard-61F7ED72
- removed kibuzzard-61F7ED8A: G***, kibuzzard-61F7ED8A
- removed kibuzzard-61F7EDAC: G***, kibuzzard-61F7EDAC
- removed kibuzzard-61F7EDC6: G***, kibuzzard-61F7EDC6
- removed kibuzzard-61F7EF48: G***, kibuzzard-61F7EF48
- removed kibuzzard-61F7EFEB: G***, kibuzzard-61F7EFEB
- removed kibuzzard-61F7FB1D: G***, kibuzzard-61F7FB1D
- removed kibuzzard-61F7FBA3: G***, kibuzzard-61F7FBA3
- removed kibuzzard-61F7FBC2: G***, kibuzzard-61F7FBC2
- removed kibuzzard-61F82282: G***, kibuzzard-61F82282
- removed kibuzzard-61F8332E: G***, kibuzzard-61F8332E
- removed kibuzzard-61F83333: G***, kibuzzard-61F83333
- removed kibuzzard-620CE59A: G***, kibuzzard-620CE59A
- removed kibuzzard-620D3625: G***, kibuzzard-620D3625
- removed kibuzzard-620D363E: G***, kibuzzard-620D363E
- removed kibuzzard-620D3646: G***, kibuzzard-620D3646
- removed kibuzzard-620D3ACF (x2): G***, kibuzzard-620D3ACF
- removed kibuzzard-620D3AFB (x2): G***, kibuzzard-620D3AFB
- removed kibuzzard-620D3FD3 (x2): G***, kibuzzard-620D3FD3
- removed kibuzzard-620D3FE5: G***, kibuzzard-620D3FE5
- removed kibuzzard-620D4024 (x2): G***, kibuzzard-620D4024
- removed kibuzzard-620D404F: G***, kibuzzard-620D404F
- removed kibuzzard-620D4F5E: G***, kibuzzard-620D4F5E
- removed kibuzzard-620D4F84: G***, kibuzzard-620D4F84
- added C7: C, Capacitor_SMD:CP_Elec_6.3x7.7, F.Cu at (94.0, 102.6)
- added J14: Conn_01x03_Male, Connector_PinHeader_2.54mm:PinHeader_1x03_P2.54mm_Vertical, F.Cu at (95.0, 116.3)
- added J15: Conn_01x03_Male, Connector_PinHeader_2.54mm:PinHeader_1x03_P2.54mm_Vertical, F.Cu at (92.4, 116.3)
- J7: value Conn_01x06_Male -> Conn_01x07_Male; footprint Connector_PinHeader_2.54mm:PinHeader_1x06_P2.54mm_Vertical -> Connector_JST:JST_EH_B7B-EH-A_1x07_P2.50mm_Vertical
- U4: value TB6612FNG -> DRV8825; footprint motor_driver:TB6612FNG_2 -> stepper_motor_driver:IC_DRV8825_STEPPER_MOTOR_DRIVER_CARRIER
- moved J7 2.11 mm to (125.0, 36.8), turned to 180 degrees
- moved U4 0.96 mm to (93.9, 107.4), turned to 180 degrees
Connections:
- J7 pad 1: /35 -> /32
- J7 pad 2: /34 -> /35
- J7 pad 3: /39 -> /34
- J7 pad 4: /36 -> /39
- J7 pad 5: GND -> /36
- J7 pad 6: /3V3 -> GND
- R11 pad 1: /32 -> /12
- T2 pad 1: /OUT1B -> /A_2
- T2 pad 2: /OUT2B -> /A_1
- T2 pad 3: /OUT3B -> /B_1
- T2 pad 4: /OUT4B -> /B_2
- U4 pad 1: /12V_P -> /13
- U4 pad 10: /3V3 -> unconnected-(U4-Pad10)
- U4 pad 11: Net-(R18-Pad2) -> /A_2
- U4 pad 12: Net-(R17-Pad2) -> /A_1
- U4 pad 13: /3V3 -> /B_1
- U4 pad 14: Net-(R15-Pad2) -> /B_2
- U4 pad 15: Net-(R16-Pad2) -> GND
- U4 pad 16: /3V3 -> /12V_P
- U4 pad 2: /3V3 -> /M0
- U4 pad 3: GND -> /M1
- U4 pad 4: /OUT1B -> /M2
- U4 pad 5: /OUT2B -> unconnected-(U4-Pad5)
- U4 pad 6: /OUT4B -> unconnected-(U4-Pad6)
- U4 pad 7: /OUT3B -> /14
- U4 pad 8: GND -> /27
Routing:
- net /27: track 110.7 -> 72.4 mm, vias 2 -> 0
- net /14: track 114.7 -> 76.9 mm, vias 2 -> 0
- net /OUT3B: track 24.4 -> 0.00 mm
- net /OUT2B: track 24.4 -> 0.00 mm
- net /12V_P: track 41.4 -> 65.1 mm
- net /33: track 87.4 -> 69.5 mm
- net /3V3: track 240.1 -> 222.8 mm
- net /26: track 89.9 -> 74.8 mm, vias 2 -> 0
- net /OUT1B: track 14.0 -> 0.00 mm
- net /A_2: track 0.00 -> 13.5 mm
- net /A_1: track 0.00 -> 12.5 mm
- net /B_2: track 0.00 -> 12.3 mm
- net /B_1: track 0.00 -> 11.5 mm
- net /OUT3A: track 23.6 -> 12.2 mm
- net /OUT2A: track 23.6 -> 12.2 mm
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Other:
- board text added: "A1"
- board text added: "A2"
- board text added: "B1"
- board text added: "B2"
- board text added: "DIR"
- board text added: "FLT"
- board text added: "GND_M"
- board text added: "M0"
- board text added: "M1"
- board text added: "M2"
- board text added: "RST"
- board text added: "SLP"
- board text added: "STEP"
- board text removed: "IN1=IN3=25, TP1 SHORT IN2=IN4=26, TP2 SHORT"
- board text removed: "IN5=IN7=12, TP3 SHORT IN6=IN8=13, TP4 SHORT"
- board text removed: "Parallel Mode"
