File: sra_dev_board_2022/sra_dev_board_2022.kicad_sch (KiCad schematic)
At the start: 77 parts, among them J1 Conn_01x19_Male, J11 Conn_01x05_Male, J12 Conn_01x05_Male, J13 Conn_01x05_Male, J2 Conn_01x03_Male, J3 Conn_01x03_Male, J4 Conn_01x03_Male, J5 Conn_01x19_Male, J6 DCJ200-10-A-XX-X_REVA, J7 Conn_01x06_Male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

Commit message: Finalised SRA Dev Board 2022 Design, added gerbers, renders, assets
Parts:
- F1: footprint Diode_THT:D_DO-15_P5.08mm_Vertical_AnodeUp -> RUEF150_3,2A_trip:RUEF160
- F2: footprint Diode_THT:D_DO-15_P5.08mm_Vertical_AnodeUp -> RXEF050_1A_trip:RXEF050
Connections:
- net 3V3: now also J9.2 (Pin_2); no longer J9.1 (Pin_1)
- net GND: now also J9.1 (Pin_1); no longer J8.6 (Pin_6), J9.2 (Pin_2)
- no-connect marks 4 -> 5
Other:
- note added: "RUEF160 PTC Resetable Fuse I_trip = 3.2A; I_hold = 1.6A"
- note added: "RXEF050 PTC Resetable Fuse I_trip = 1A; I_hold = 0.5A"
Changed lines of the file:
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@@
   (no_connect (at 176.784 114.681))
   (no_connect (at 118.0338 114.8334))
+  (no_connect (at 162.5092 175.133))
   (no_connect (at 118.0338 104.6734))
   (no_connect (at 176.784 104.521))
@@
     (stroke (width 0) (type default) (color 0 0 0 0))
   )
-  (wire (pts (xy 178.2318 133.1468) (xy 171.7294 133.1468))
+  (wire (pts (xy 146.431 104.2162) (xy 139.9286 104.2162))
     (stroke (width 0) (type default) (color 0 0 0 0))
   )
@@
     (effects (font (size 2 2) (thickness 0.6) bold) (justify left bottom))
   )
+  (text "RXEF050 PTC Resetable Fuse \nI_trip = 1A; I_hold = 0.5A"
+    (at 161.7472 134.3914 0)
+    (effects (font (size 1.2 1.2) bold) (justify left bottom))
+  )
   (text "Mounting Holes" (at 98.9076 209.296 0)
     (effects (font (size 2 2) (thickness 0.6) bold) (justify left bottom))
@@
   )
   (text "12V_U: Raw Input 12V\n12V_P: 12V with protection circuit"
-    (at 75.7428 128.016 0)
+    (at 74.0664 128.8796 0)
     (effects (font (size 1.5 1.5) bold) (justify left bottom))
   )
@@
     (effects (font (size 2 2) (thickness 0.6) bold) (justify left bottom))
   )
+  (text "RUEF160 PTC Resetable Fuse \nI_trip = 3.2A; I_hold = 1.6A"
+    (at 103.0986 134.4422 0)
+    (effects (font (size 1.2 1.2) bold) (justify left bottom))
+  )
   (text "LM2576: Buck Regulator" (at 132.842 22.86 0)
     (effects (font (size 2 2) (thickness 0.6) bold) (justify left bottom))
@@
     (effects (font (size 2 2) (thickness 0.6) bold) (justify left bottom))
   )
-  (text "1N5822 <=> SS34 (3A \nSchottky diode)" (at 74.676 133.35 0)
+  (text "1N5822 <=> SS34 \n(3A Schottky diode)" (at 74.0664 134.366 0)
     (effects (font (size 1.2 1.2) bold) (justify left bottom))
   )
@@
     (effects (font (size 1.27 1.27)) (justify left bottom))
   )
-  (label "AMS_IN" (at 178.2318 133.1468 0)
+  (label "AMS_IN" (at 146.431 104.2162 0)
     (effects (font (size 1.27 1.27)) (justify left bottom))
   )
-  (label "3V3" (at 144.8054 218.567 0)
+  (label "3V3" (at 144.8054 221.107 0)
     (effects (font (size 1.27 1.27)) (justify left bottom))
   )
@@
     (effects (font (size 1.27 1.27)) (justify left bottom))
   )
-  (label "GND" (at 144.8054 221.107 0)
+  (label "GND" (at 144.8054 218.567 0)
     (effects (font (size 1.27 1.27)) (justify left bottom))
   )
@@
     (effects (font (size 1.27 1.27)) (justify left bottom))
   )
-  (label "5V_P" (at 171.7294 133.1468 180)
+  (label "5V_P" (at 139.9286 104.2162 180)
     (effects (font (size 1.27 1.27)) (justify right bottom))
   )
@@
     (effects (font (size 1.27 1.27)) (justify right bottom))
   )
-  (label "GND" (at 162.5092 175.133 180)
-    (effects (font (size 1.27 1.27)) (justify right bottom))
-  )
   (label "27" (at 54.9402 152.9842 180)
     (effects (font (size 1.27 1.27)) (justify right bottom))
@@
     (property "Reference" "F1" (id 0) (at 97.028 109.474 90))
     (property "Value" "3A" (id 1) (at 97.2058 114.9604 90))
-    (property "Footprint" "Diode_THT:D_DO-15_P5.08mm_Vertical_AnodeUp" (id 2) (at 97.1296 113.792 90)
+    (property "Footprint" "RUEF150_3,2A_trip:RUEF160" (id 2) (at 97.1296 113.792 90)
       (effects (font (size 1.27 1.27)) hide)
     )
@@
     (property "Reference" "F2" (id 0) (at 155.6766 109.0168 90))
     (property "Value" "300mA" (id 1) (at 156.1846 114.6556 90))
-    (property "Footprint" "Diode_THT:D_DO-15_P5.08mm_Vertical_AnodeUp" (id 2) (at 155.8798 113.6396 90)
+    (property "Footprint" "RXEF050_1A_trip:RXEF050" (id 2) (at 155.8798 113.6396 90)
       (effects (font (size 1.27 1.27)) hide)
     )
@@
     )
     (path "/7fc6eda3-a41a-4ab9-935d-37e18cb30594"
-      (reference "F1") (unit 1) (value "3A") (footprint "Diode_THT:D_DO-15_P5.08mm_Vertical_AnodeUp")
+      (reference "F1") (unit 1) (value "3A") (footprint "RUEF150_3,2A_trip:RUEF160")
     )
     (path "/a0e1d03b-10bf-47bf-bb19-34f370c33a49"
-      (reference "F2") (unit 1) (value "300mA") (footprint "Diode_THT:D_DO-15_P5.08mm_Vertical_AnodeUp")
+      (reference "F2") (unit 1) (value "300mA") (footprint "RXEF050_1A_trip:RXEF050")
     )
     (path "/f830bcd1-bd58-489f-a51a-00a07fc7d5b6"

Commit message: SRA Board, MPU, LSA Kicad, Gerber files updated
Parts:
- added J10: Conn_01x03_Male, pin_header_connectors:1X03, symbol Connector:Conn_01x03_Male
Connections:
- net 15: now also J10.1 (Pin_1)
- net 16: no longer SW4.2
- net 17: no longer SW3.2
- net 2: no longer SW2.2
- net 4: no longer SW1.2
- net 5V: now also J10.2 (Pin_2)
- net GND: now also SW1.2, SW2.2, SW3.2, SW4.2, J10.3 (Pin_3); no longer SW1.3, SW2.3, SW3.3, SW4.3
- no-connect marks 5 -> 9
Other:
- moved on the sheet: J2, J3, J4

Commit message: add DRV8825 Stepper Driver
Parts:
- removed J7: Conn_01x06_Male, Connector_PinHeader_2.54mm:PinHeader_1x06_P2.54mm_Vertical, symbol Connector:Conn_01x06_Male
- removed R15, R16, R17, R18: 1k, Resistor_SMD:R_1206_3216Metric, symbol Device:R
- removed TB_A1, TB_B1: SW_Push_DPDT, dpdt_tht:dpdt_sw_2x03_tht, symbol Switch:SW_Push_DPDT
- removed TP1, TP2, TP3, TP4: TestPoint, testpoint_pad:pad_1,27-2,54_smd, symbol Connector:TestPoint
- removed U4: TB6612FNG, motor_driver:TB6612FNG_2, symbol TB6612FNG:ROB-14450
- added C7: C, Capacitor_SMD:CP_Elec_6.3x7.7, symbol Device:C_Polarized_Small
- added J14, J15: Conn_01x03_Male, Connector_PinHeader_2.54mm:PinHeader_1x03_P2.54mm_Vertical, symbol Connector:Conn_01x03_Male
- added J7: Conn_01x07_Male, Connector_JST:JST_EH_B7B-EH-A_1x07_P2.50mm_Vertical, symbol Connector:Conn_01x07_Male
- added U4: DRV8825, stepper_motor_driver:IC_DRV8825_STEPPER_MOTOR_DRIVER_CARRIER, symbol DRV8825_STEPPER_MOTOR_DRIVER_CARRIER:DRV8825_STEPPER_MOTOR_DRIVER_CARRIER
Connections:
- net 12: now also R11.1
- net 12V_P: now also C7.1, U4.16 (VMOT)
- net 13: now also U4.1 (~{EN})
- net 14: now also U4.7 (STEP)
- net 27: now also U4.8 (DIR)
- net 32: now also J7.1 (Pin_1); no longer R11.1
- net 34: now also J7.3 (Pin_3)
- net 35: now also J7.2 (Pin_2)
- net 36: now also J7.5 (Pin_5)
- net 39: now also J7.4 (Pin_4)
- net 3V3: now also J15.1 (Pin_1), J15.2 (Pin_2), J15.3 (Pin_3), J7.7 (Pin_7)
- net GND: now also C7.2, J7.6 (Pin_6), U4.15 (GND_MOT), U4.9 (GND)
- net OUT1B renamed A_2
- net A_2: now also U4.11 (A2)
- net OUT2B renamed A_1
- net A_1: now also U4.12 (A1)
- net OUT3B renamed B_1
- net B_1: now also U4.13 (B1)
- net OUT4B renamed B_2
- net B_2: now also U4.14 (B2)
- new net M0: J14.1 (Pin_1), U4.2 (M0)
- new net M1: J14.2 (Pin_2), U4.3 (M1)
- new net M2: J14.3 (Pin_3), U4.4 (M2)
- no-connect marks 9 -> 12
Other:
- note added: "DRV8825"
- note added: "STEPPER DRIVER"
- note added: "connect jumpers for microstepping"
- note removed: "Motor Normal-Parallel Mode"
- note removed: "Motor Output Pins"
- note removed: "TESTPOINTS"
- moved on the sheet: 12V_SW1, 5V_SW1, D13, D9, F1, F2, R11, R12, R13, R14, SW1, SW2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
