File: sra_dev_board_2022/sra_dev_board_2022.kicad_sch (KiCad schematic)
At the start: 78 parts, among them J1 Conn_01x19_Male, J10 Conn_01x03_Male, J11 Conn_01x05_Male, J12 Conn_01x05_Male, J13 Conn_01x05_Male, J2 Conn_01x03_Male, J3 Conn_01x03_Male, J4 Conn_01x03_Male, J5 Conn_01x19_Male, J6 DCJ200-10-A-XX-X_REVA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

Commit message: Add footprint and symbol for DRV8825 and update schematic
Parts:
- removed J7: Conn_01x06_Male, Connector_PinHeader_2.54mm:PinHeader_1x06_P2.54mm_Vertical, symbol Connector:Conn_01x06_Male
- removed R15, R16, R17, R18: 1k, Resistor_SMD:R_1206_3216Metric, symbol Device:R
- removed TB_B1: SW_Push_DPDT, dpdt_tht:dpdt_sw_2x03_tht, symbol Switch:SW_Push_DPDT
- removed TP3, TP4: TestPoint, testpoint_pad:pad_1,27-2,54_smd, symbol Connector:TestPoint
- removed U4: TB6612FNG, motor_driver:TB6612FNG_2, symbol TB6612FNG:ROB-14450
- added C7: 100uF, Capacitor_SMD:CP_Elec_6.3x7.7, symbol Device:C_Polarized_Small_US
- added J14, J15: Conn_01x03_Male, Connector_PinHeader_2.54mm:PinHeader_1x03_P2.54mm_Vertical, symbol Connector:Conn_01x03_Male
- added J7: Conn_01x07_Male, Connector_PinHeader_2.54mm:PinHeader_1x07_P2.54mm_Vertical, symbol Connector:Conn_01x07_Male
- added U4: DRV8825_STEPPER_MOTOR_DRIVER_CARRIER, stepper_motor_driver:IC_DRV8825_STEPPER_MOTOR_DRIVER_CARRIER, symbol DRV8825_STEPPER_MOTOR_DRIVER_CARRIER:DRV8825_STEPPER_MOTOR_DRIVER_CARRIER
Connections:
- net 12: now also D1.2 (A), R11.1, TB_A1.1 (A), TB_A1.2 (B); no longer D7.2 (A)
- net 12V_P: now also C7.1, U4.16 (VMOT)
- net 13: now also D7.2 (A), U4.1 (~{EN}); no longer D8.2 (A)
- net 14: now also U4.7 (STEP)
- net 25: now also TB_A1.4 (A); no longer TB_A1.3 (C)
- net 27: now also U4.8 (DIR)
- net 32: now also D8.2 (A), J7.1 (Pin_1); no longer D1.2 (A), R11.1, TB_A1.1 (A), TB_A1.2 (B)
- net 33: now also TB_A1.3 (C); no longer TB_A1.4 (A)
- net 34: now also J7.3 (Pin_3)
- net 35: now also J7.2 (Pin_2)
- net 36: now also J7.5 (Pin_5)
- net 39: now also J7.4 (Pin_4)
- net 3V3: now also J15.1 (Pin_1), J15.2 (Pin_2), J15.3 (Pin_3), J7.7 (Pin_7)
- net GND: now also C7.2, J7.6 (Pin_6), U4.15 (GND_MOT), U4.9 (GND)
- net OUT1B renamed A_1
- net A_1: now also U4.12 (A1)
- net OUT2B renamed A_2
- net A_2: now also U4.11 (A2)
- net OUT3B renamed B_1
- net B_1: now also U4.13 (B1)
- net OUT4B renamed B_2
- net B_2: now also U4.14 (B2)
- new net M0: J14.1 (Pin_1), U4.2 (M0)
- new net M1: J14.2 (Pin_2), U4.3 (M1)
- new net M2: J14.3 (Pin_3), U4.4 (M2)
- no-connect marks 9 -> 12
Other:
- note added: "DRV8825"
- note added: "MOTOR DRIVERS"
- note removed: "MOTOR DRIVER"
- moved on the sheet: 12V_SW1, 5V_SW1, D13, D9, F1, F2, R11, R12, R13, R14, SW1, SW2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

Commit message: Modify routing according to new schematic
Connections:
- net 25: now also TB_A1.3 (C); no longer TB_A1.4 (A)
- net 33: now also TB_A1.4 (A); no longer TB_A1.3 (C)
- net A_1: now also T2.2 (Pin_2); no longer T2.1 (Pin_1)
- net A_2: now also T2.1 (Pin_1); no longer T2.2 (Pin_2)
Changed lines of the file:
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@@
     (effects (font (size 1.27 1.27)) (justify left bottom))
   )
-  (label "A_1" (at 259.4102 29.6164 0)
+  (label "A_2" (at 259.4102 29.6164 0)
     (effects (font (size 1.27 1.27)) (justify left bottom))
   )
@@
     (effects (font (size 1.27 1.27)) (justify right bottom))
   )
-  (label "33" (at 46.9392 114.3 180)
+  (label "25" (at 46.9392 114.3 180)
     (effects (font (size 1.27 1.27)) (justify right bottom))
   )
@@
     (effects (font (size 1.27 1.27)) (justify right bottom))
   )
-  (label "A_2" (at 259.4102 32.1564 0)
+  (label "A_1" (at 259.4102 32.1564 0)
     (effects (font (size 1.27 1.27)) (justify left bottom))
   )
@@
     (effects (font (size 1.27 1.27)) (justify left bottom))
   )
-  (label "25" (at 46.9392 119.38 180)
+  (label "33" (at 46.9392 119.38 180)
     (effects (font (size 1.27 1.27)) (justify right bottom))
   )
