File: sensors_2022/lsa/lsa/lsa.kicad_pcb (KiCad board)
At the start: 2 copper layers, 61.7 x 22.7 mm, 29 parts, among them J1 Conn_01x06_Male, U1 LM324

Commit message: SRA Board, MPU, LSA Kicad, Gerber files updated
Parts:
- added REF**: MountingHole_3.2mm_M3, MountingHole:MountingHole_3.2mm_M3, F.Cu at (98.5, 88.2)
- added REF**: MountingHole_3.2mm_M3, MountingHole:MountingHole_3.2mm_M3, F.Cu at (133.9, 88.2)
- moved D4 2.55 mm to (144.1, 88.2), turned to 180 degrees
- moved D2 2.54 mm to (108.6, 88.2), turned to 180 degrees
- moved R7 2.17 mm to (129.4, 79.7)
- moved R3 2.12 mm to (129.4, 88.2)
- moved R5 1.81 mm to (93.9, 79.7)
- moved R1 1.76 mm to (93.9, 88.2)
- moved R2 1.73 mm to (102.9, 88.2)
- moved R6 1.72 mm to (102.9, 79.7)
- moved R4 1.71 mm to (138.4, 88.2)
- moved R8 1.69 mm to (138.4, 79.7)
Routing:
- net +3V3: track 195.9 -> 169.9 mm
- net GND: track 64.5 -> 59.0 mm
- net Net-(D2-Pad1): track 5.49 -> 9.88 mm
- net /LSA_A0: track 13.8 -> 11.6 mm
- net Net-(D3-Pad1): track 5.88 -> 3.76 mm
- net Net-(D1-Pad1): track 5.50 -> 3.74 mm
- net /LSA_A3: track 13.4 -> 11.7 mm
- net Net-(D4-Pad1): track 5.50 -> 6.33 mm
- net /LSA_A2: track 26.8 -> 26.1 mm
