File: sensors_2023/mpu/mpu/mpu.kicad_pcb (KiCad board)
At the start: 2 copper layers, 22 x 13 mm, 4 parts, among them J1 Conn_01x06_Male, J2 Conn_01x08_Female

Commit message: Updated working content for sra_dev_board_2023
Parts:
- added kibuzzard-637B8032: G***, kibuzzard-637B8032, F.Cu at (151.9, 75.0)
Routing:
- net /GND: track 17.2 -> 1.23 mm
- net /3V3: track 24.2 -> 23.0 mm
