File: sra_dev_board_2023/sra_dev_board_2023.kicad_pcb (KiCad board)
At the start: 2 copper layers, 81.2 x 92.7 mm, 200 parts, among them J1 Conn_01x19_Male, J10 Conn_01x03_Male, J11 Conn_01x05_Male, J12 Conn_01x05_Male, J13 Conn_01x05_Male, J14 Conn_01x03_Male, J15 Conn_01x03_Male, J16 Screw_Terminal_01x05, J17 Conn_01x06_Male, J2 Conn_01x03_Male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

Commit message: Add current limiting resistor for MPU (#26)
* Add current limiting resistor on Interrupt line for MPU

* Update gerbers, placement files and BoM
Parts:
- removed kibuzzard-637A0F99: G***, kibuzzard-637A0F99
- added R15: 4.7k, Resistor_SMD:R_0603_1608Metric, F.Cu at (137.5, 45.1)
- added kibuzzard-63F471C8: G***, kibuzzard-63F471C8, F.Cu at (126.5, 42.3)
- moved kibuzzard-61F7D60F 18.7 mm to (120.3, 40.8), turned to 0 degrees
Connections:
- J8 pad 4: /23 -> Net-(J8-Pad4)
Routing:
- net /23: track 97.6 -> 85.8 mm
- net Net-(J8-Pad4): track 0.00 -> 8.76 mm, vias 0 -> 1
